Commit message: modify my_robot
modify my_robot chassis, change the length to 0.15 so it won't generate friction.

File: catkim_ws/src/my_robot/urdf/my_robot.xacro (robot description, xacro)
@@ -22,5 +22,5 @@
       <origin xyz="0 0 0" rpy=" 0 0 0"/>
       <geometry>
-        <cylinder radius="0.2" length="0.2"/>
+        <cylinder radius="0.2" length="0.15"/>
       </geometry>
     </collision>
@@ -28,5 +28,5 @@
       <origin xyz="0 0 0" rpy=" 0 0 0"/>
       <geometry>
-        <cylinder radius="0.2" length="0.2"/>
+        <cylinder radius="0.2" length="0.15"/>
       </geometry>
     </visual>
